Commit message: change urdf

File: description/camera.xacro (robot description, xacro)
@@ -4,5 +4,5 @@
         <parent link="chassis" />
         <child link="camera_link" />
-        <origin xyz="0.305 0 0.25" rpy="0 0 0"/>
+        <origin xyz="0.405 0 0.25" rpy="0 0 0"/>
     </joint>
     <link name="camera_link">

File: description/lidar.xacro (robot description, xacro)
@@ -4,5 +4,5 @@
         <parent link="chassis" />
         <child link="laser_frame" />
-        <origin xyz="0.1 0 0.325" rpy="0 0 0"/>
+        <origin xyz="0.175 0 0.325" rpy="0 0 0"/>
     </joint>
     <link name="laser_frame">

File: description/robot_core.xacro (robot description, xacro)
@@ -2,5 +2,8 @@
 <robot xmlns:xacro="http://www.ros.org/wiki/xacro"  name="robot">
     <xacro:include filename="inertial_macros.xacro" />
+    <xacro:property name="chassis_length" value="0.4"/>
     <xacro:property name="wheel_thickness" value="0.01"/>
+    <xacro:property name="wheel_offset_y" value="0.1625"/>
+    <xacro:property name="wheel_radius" value="0.03375"/>
     <material name="white">
         <color rgba="1 1 1 1"/>
@@ -25,18 +28,18 @@
     <link name="chassis">
         <visual>
-            <origin xyz="0.15 0 0.15" rpy="0 0 0"/>
+            <origin xyz="${chassis_length/2} 0 0.15" rpy="0 0 0"/>
             <geometry>
-                <box size="0.3 0.3 0.3"/>
+                <box size="${chassis_length} 0.3 0.3"/>
             </geometry>
             <material name="black"/>
         </visual>
         <collision>
-            <origin xyz="0.15 0 0.15" rpy="0 0 0"/>
+            <origin xyz="${chassis_length/2} 0 0.15" rpy="0 0 0"/>
             <geometry>
-                <box size="0.3 0.3 0.3"/>
+                <box size="${chassis_length} 0.3 0.3"/>
             </geometry>
         </collision>
-        <xacro:inertial_box mass="1.0" x="0.3" y="0.3" z="0.3">
-            <origin xyz="0.15 0 0.15" rpy="0 0 0"/>
+        <xacro:inertial_box mass="1.0" x="${chassis_length}" y="0.3" z="0.3">
+            <origin xyz="${chassis_length/2} 0 0.15" rpy="0 0 0"/>
         </xacro:inertial_box>
     </link>
@@ -48,5 +51,5 @@
         <parent link="base_link"/>
         <child link="left_wheel"/>
-        <origin xyz="0 0.175 0" rpy="-${pi/2} 0 0"/>
+        <origin xyz="0 ${wheel_offset_y} 0" rpy="-${pi/2} 0 0"/>
         <axis xyz="0 0 1"/>
     </joint>
@@ -54,5 +57,5 @@
         <visual>
             <geometry>
-                <cylinder length="${wheel_thickness}" radius="0.05" />
+                <cylinder length="${wheel_thickness}" radius="${wheel_radius}" />
             </geometry>
             <material name="blue"/>
@@ -60,8 +63,8 @@
         <collision>
             <geometry>
-                <cylinder length="${wheel_thickness}" radius="0.05" />
+                <cylinder length="${wheel_thickness}" radius="${wheel_radius}" />
             </geometry>
         </collision>
-        <xacro:inertial_cylinder mass="0.1" length="${wheel_thickness}" radius="0.05">
+        <xacro:inertial_cylinder mass="0.05" length="${wheel_thickness}" radius="${wheel_radius}">
             <origin xyz="0 0 0" rpy="0 0 0"/>
         </xacro:inertial_cylinder>
@@ -74,5 +77,5 @@
         <parent link="base_link"/>
         <child link="right_wheel"/>
-        <origin xyz="0 -0.175 0" rpy="${pi/2} 0 0"/>
+        <origin xyz="0 ${-wheel_offset_y} 0" rpy="${pi/2} 0 0"/>
         <axis xyz="0 0 -1"/>
     </joint>
@@ -80,5 +83,5 @@
         <visual>
             <geometry>
-                <cylinder length="${wheel_thickness}" radius="0.05" />
+                <cylinder length="${wheel_thickness}" radius="${wheel_radius}" />
             </geometry>
             <material name="blue"/>
@@ -86,8 +89,8 @@
         <collision>
             <geometry>
-                <cylinder length="${wheel_thickness}" radius="0.05" />
+                <cylinder length="${wheel_thickness}" radius="${wheel_radius}" />
             </geometry>
         </collision>
-        <xacro:inertial_cylinder mass="0.1" length="${wheel_thickness}" radius="0.05">
+        <xacro:inertial_cylinder mass="0.05" length="${wheel_thickness}" radius="${wheel_radius}">
             <origin xyz="0 0 0" rpy="0 0 0"/>
         </xacro:inertial_cylinder>
@@ -100,10 +103,10 @@
         <parent link="chassis"/>
         <child link="caster_wheel"/>
-        <origin xyz="0.24 0 0" rpy="0 0 0"/>
+        <origin xyz="0.3 0 0" rpy="0 0 0"/>
     </joint>
     <link name="caster_wheel">
         <visual>
             <geometry>
-                <sphere radius="0.05" />
+                <sphere radius="0.03" />
             </geometry>
             <material name="white"/>
@@ -111,8 +114,8 @@
         <collision>
             <geometry>
-                <sphere radius="0.05" />
+                <sphere radius="0.03" />
             </geometry>
         </collision>
-        <xacro:inertial_sphere mass="0.1" radius="0.05">
+        <xacro:inertial_sphere mass="0.01" radius="0.03">
             <origin xyz="0 0 0" rpy="0 0 0"/>
         </xacro:inertial_sphere>
