Commit message: launch real robot control

File: description/gazebo_control.xacro (robot description, xacro)
@@ -6,6 +6,6 @@
             <left_joint>left_wheel_joint</left_joint>
             <right_joint>right_wheel_joint</right_joint>
-            <wheel_separation>0.35</wheel_separation>
-            <wheel_diameter>0.1</wheel_diameter>
+            <wheel_separation>0.335</wheel_separation>
+            <wheel_diameter>0.068</wheel_diameter>
             <!-- Limits -->
             <max_wheel_torque>200</max_wheel_torque>

File: description/robot_core.xacro (robot description, xacro)
@@ -4,6 +4,6 @@
     <xacro:property name="chassis_length" value="0.4"/>
     <xacro:property name="wheel_thickness" value="0.01"/>
-    <xacro:property name="wheel_offset_y" value="0.1625"/>
-    <xacro:property name="wheel_radius" value="0.03375"/>
+    <xacro:property name="wheel_offset_y" value="0.1675"/>
+    <xacro:property name="wheel_radius" value="0.034"/>
     <material name="white">
         <color rgba="1 1 1 1"/>

File: description/ros2_control.xacro (robot description, xacro)
@@ -1,7 +1,35 @@
 <?xml version="1.0"?>
 <robot xmlns:xacro="http://www.ros.org/wiki/xacro">
-    <ros2_control name="GazeboSystem" type="system">
+    <!-- <ros2_control name="GazeboSystem" type="system">
         <hardware>
             <plugin>gazebo_ros2_control/GazeboSystem</plugin>
+        </hardware>
+        <joint name="left_wheel_joint">
+            <command_interface name="velocity">
+                <param name="min">-10</param>
+                <param name="max">10</param>
+            </command_interface>
+            <state_interface name="velocity" />
+            <state_interface name="position" />
+        </joint>
+        <joint name="right_wheel_joint">
+            <command_interface name="velocity">
+                <param name="min">-10</param>
+                <param name="max">10</param>
+            </command_interface>
+            <state_interface name="velocity" />
+            <state_interface name="position" />
+        </joint>
+    </ros2_control> -->
+    <ros2_control name="RealRobot" type="system">
+        <hardware>
+            <plugin>diffdrive_arduino/DiffDriveArduino</plugin>
+            <param name="left_wheel_name">left_wheel_joint</param>
+            <param name="right_wheel_name">right_wheel_joint</param>
+            <param name="loop_rate">30</param>
+            <param name="device">/dev/serial/by-path/platform-fd500000.pcie-pci-0000:01:00.0-usb-0:1.2:1.0-port0</param>
+            <param name="baud_rate">57600</param>
+            <param name="timeout">1000</param>
+            <param name="enc_counts_per_rev">1500</param>
         </hardware>
         <joint name="left_wheel_joint">
