Commit message: basic gazebo sim and control

File: description/robot_core.xacro (robot description, xacro)
@@ -37,4 +37,7 @@
         </xacro:inertial_box>
     </link>
+    <gazebo reference="chassis">
+        <material>Gazebo/Black</material>
+    </gazebo>
     <!-- Left wheel link -->
     <joint name="left_wheel_joint" type="continuous">
@@ -60,4 +63,7 @@
         </xacro:inertial_cylinder>
     </link>
+    <gazebo reference="left_wheel">
+        <material>Gazebo/Blue</material>
+    </gazebo>
     <!-- Right wheel link -->
     <joint name="right_wheel_joint" type="continuous">
@@ -83,4 +89,7 @@
         </xacro:inertial_cylinder>
     </link>
+    <gazebo reference="right_wheel">
+        <material>Gazebo/Blue</material>
+    </gazebo>
     <!-- CASTER WHEEL -->
     <joint name="caster_wheel_joint" type="fixed">
@@ -105,3 +114,8 @@
         </xacro:inertial_sphere>
     </link>
+    <gazebo reference="caster_wheel">
+        <material>Gazebo/Blue</material>
+        <mu1 value="0.001" />
+        <mu2 value="0.002" />
+    </gazebo>
 </robot>

Commit message: lidar urdf stuff

File: description/robot_core.xacro (robot description, xacro)
@@ -10,4 +10,7 @@
     <material name="black">
         <color rgba="0 0 0 1"/>
+    </material>
+    <material name="red">
+        <color rgba="1 0 0 1"/>
     </material>
     <link name="base_link">
@@ -117,5 +120,5 @@
         <material>Gazebo/Blue</material>
         <mu1 value="0.001" />
-        <mu2 value="0.002" />
+        <mu2 value="0.001" />
     </gazebo>
 </robot>

Commit message: slam & launch changes

File: description/robot_core.xacro (robot description, xacro)
@@ -18,5 +18,14 @@
         <color rgba="1 0 0 1"/>
     </material>
+    <!-- Base link -->
     <link name="base_link">
+    </link>
+    <!-- Base footprint link -->
+    <joint name="base_footprint_joint" type="fixed">
+        <parent link="base_link" />
+        <child link="base_footprint" />
+        <origin xyz="0 0 0" rpy="0 0 0" />
+    </joint>
+    <link name="base_footprint">
     </link>
     <!-- Chassis link -->
